File: src/KiCad/PlutoDX_PowerSupply.kicad_sch (KiCad schematic)
At the start: 21 parts, among them J1 USB_C_Receptacle_PowerOnly_6P, U1 CH224K, U2 TPS563200, U3 TPS563200

Commit message: Switch to TPS565208 from TPS563200 for better current margins
Also fix an overvoltage issue by connecting the CH224K's CFG pins to VDD instead of VBUS

Also add KiCad gitignore
Parts:
- removed U2, U3: TPS563200, Package_TO_SOT_SMD:SOT-23-6, symbol Regulator_Switching:TPS563200
- added U2, U3: TPS565208, Package_TO_SOT_SMD:SOT-23-6, symbol Regulator_Switching:TPS565208
- C1: value 1uF -> 25v 10uF
- C2, C5: value 10uF -> 25v 10uF
- F1: value Polyfuse 4A -> Polyfuse 5A
- renumbered MPLCG0530L2R3 to MPLCG0530L2R2
Connections:
- net +15V: now also U2.3 (VIN), U2.5 (EN), U3.3 (VIN), U3.5 (EN)
- net GND: now also U2.1 (GND), U3.1 (GND)
- net at C3.1, MPLCG0530L2R2.1: now also U2.2 (SW)
- net at R3.2, R4.1: now also U2.4 (VFB)
- net at C3.2: now also U2.6 (VBST)
- net at R5.1, R6.2: now also U3.4 (VFB)
- net at C6.1, MPLCG0530L2R2.1: now also U3.2 (SW)
- net at C6.2: now also U3.6 (VBST)
Other:
- moved on the sheet: C1, C2, C5
